File: hw/schematics/pcb_final_v2.kicad_sch (KiCad schematic)
At the start: 26 parts, among them J1 pin_socket-bluepill, J10 tcrt5000_conector_2, J11 tcrt5000_conector_3, J12 tcrt5000_conector_1, J2 pin_socket-bluepill, J9 tof-connector_3, SW2 key, U1 YAAJ_BluePill, U2 Receptor IR, U4 AMS1117-3.3

Commit message: Arquivo pcb_final_v2 atualizado
Connections:
- net +7.4V: no longer 7.4V1.1 (Pin_1), 7.4V1.2 (Pin_2), C2.2, C_polarized1.2, D1.2 (A), IN_buck-7.4V1.2 (Pin_2), U4.1 (GND), power_drive1.2 (Pin_2)
- new net: 7.4V1.1 (Pin_1), D1.2 (A)
- new net GNDPWR: 7.4V1.2 (Pin_2), C2.2, C_polarized1.2, IN_buck-7.4V1.2 (Pin_2), U4.1 (GND), power_drive1.2 (Pin_2)
Other:
- moved on the sheet: power_drive1
